File: Lab4/sch/Lab4Schematic/Lab4Schematic.kicad_sch (KiCad schematic)
At the start: 3 parts, among them SW1 SW_Push, U1 Pico, U2 2478

Commit message: lab 5 start
Connections:
- net at U2.23 (3V0), U2.36 (IM1), U2.37 (IM2): now also U2.38 (IM3); no longer U2.35 (IM0)
Changed lines of the file:
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@@
     (comment 2 "Maurice Otieno")
   )
-  (junction (at 151.13 98.425) (diameter 0) (color 0 0 0 0)
-  )
-  (junction (at 151.13 95.885) (diameter 0) (color 0 0 0 0)
+  (junction (at 151.13 93.345) (diameter 0) (color 0 0 0 0)
   )
   (wire (pts (xy 114.935 107.315) (xy 137.795 107.315))
@@
     (stroke (width 0) (type default))
   )
-  (wire (pts (xy 145.415 98.425) (xy 151.13 98.425))
+  (wire (pts (xy 151.13 90.805) (xy 151.13 93.345))
     (stroke (width 0) (type default))
   )
@@
     (stroke (width 0) (type default))
   )
-  (wire (pts (xy 151.13 95.885) (xy 151.13 98.425))
-    (stroke (width 0) (type default))
-  )
   (wire (pts (xy 149.225 122.555) (xy 114.935 122.555))
     (stroke (width 0) (type default))
@@
   )
   (wire (pts (xy 140.335 106.045) (xy 140.335 112.395))
+    (stroke (width 0) (type default))
+  )
+  (wire (pts (xy 145.415 93.345) (xy 151.13 93.345))
     (stroke (width 0) (type default))
   )
@@
     (stroke (width 0) (type default))
   )
-  (wire (pts (xy 145.415 128.905) (xy 145.415 98.425))
+  (wire (pts (xy 145.415 128.905) (xy 145.415 93.345))
     (stroke (width 0) (type default))
   )
